Commit message: added new Mass

File: mqp_ws/src/franka_description/robots/hand.xacro (robot description, xacro)
@@ -21,5 +21,5 @@
       </collision>
 	<inertial>
-            <mass value="0.1" />
+            <mass value="0.67893" />
             <inertia ixx="0.03" iyy="0.03" izz="0.03" ixy="0.0" ixz="0.0" iyz="0.0" />
         </inertial>
@@ -37,5 +37,5 @@
       </collision>
 	<inertial>
-            <mass value="0.1" />
+            <mass value="0.01053" />
             <inertia ixx="0.03" iyy="0.03" izz="0.03" ixy="0.0" ixz="0.0" iyz="0.0" />
         </inertial>
@@ -55,5 +55,5 @@
       </collision>
 	<inertial>
-            <mass value="0.1" />
+            <mass value="0.01053" />
             <inertia ixx="0.03" iyy="0.03" izz="0.03" ixy="0.0" ixz="0.0" iyz="0.0" />
         </inertial>

File: mqp_ws/src/franka_description/robots/panda_arm.xacro (robot description, xacro)
@@ -26,5 +26,5 @@
       </collision>
       <inertial>
-        <mass value="0.1" />
+        <mass value="3.06357" />
         <inertia ixx="0.03" iyy="0.03" izz="0.03" ixy="0.0" ixz="0.0" iyz="0.0" />
       </inertial>
@@ -42,5 +42,5 @@
       </collision>
       <inertial>
-        <mass value="0.1" />
+        <mass value="2.34471" />
         <inertia ixx="0.03" iyy="0.03" izz="0.03" ixy="0.0" ixz="0.0" iyz="0.0" />
       </inertial>
@@ -66,5 +66,5 @@
       </collision>
       <inertial>
-        <mass value="0.1" />
+        <mass value="2.36414" />
         <inertia ixx="0.03" iyy="0.03" izz="0.03" ixy="0.0" ixz="0.0" iyz="0.0" />
       </inertial>
@@ -90,5 +90,5 @@
       </collision>
       <inertial>
-        <mass value="0.1" />
+        <mass value="2.38050" />
         <inertia ixx="0.03" iyy="0.03" izz="0.03" ixy="0.0" ixz="0.0" iyz="0.0" />
       </inertial>
@@ -114,5 +114,5 @@
       </collision>
       <inertial>
-        <mass value="0.1" />
+        <mass value="2.42754" />
         <inertia ixx="0.03" iyy="0.03" izz="0.03" ixy="0.0" ixz="0.0" iyz="0.0" />
       </inertial>
@@ -138,5 +138,5 @@
       </collision>
       <inertial>
-        <mass value="0.1" />
+        <mass value="3.49611" />
         <inertia ixx="0.03" iyy="0.03" izz="0.03" ixy="0.0" ixz="0.0" iyz="0.0" />
       </inertial>
@@ -162,5 +162,5 @@
       </collision>
       <inertial>
-        <mass value="0.1" />
+        <mass value="1.46736" />
         <inertia ixx="0.03" iyy="0.03" izz="0.03" ixy="0.0" ixz="0.0" iyz="0.0" />
       </inertial>
@@ -186,5 +186,5 @@
       </collision>
       <inertial>
-        <mass value="0.1" />
+        <mass value="0.45606" />
         <inertia ixx="0.03" iyy="0.03" izz="0.03" ixy="0.0" ixz="0.0" iyz="0.0" />
       </inertial>
