Commit message: added colors?

File: mqp_ws/src/franka_description/robots/panda_arm.xacro (robot description, xacro)
@@ -277,32 +277,40 @@
     </transmission>
     <gazebo reference="${arm_id}_link0">
+      <material>Gazebo/White</material>
       <mu1>0.61</mu1>
       <mu2>0.61</mu2>
     </gazebo>
     <gazebo reference="${arm_id}_link1">
+      <material>Gazebo/White</material>
       <mu1>0.61</mu1>
       <mu2>0.61</mu2>
     </gazebo>
     <gazebo reference="${arm_id}_link2">
+      <material>Gazebo/White</material>
       <mu1>0.61</mu1>
       <mu2>0.61</mu2>
     </gazebo>
     <gazebo reference="${arm_id}_link3">
+      <material>Gazebo/White</material>
       <mu1>0.61</mu1>
       <mu2>0.61</mu2>
     </gazebo>
     <gazebo reference="${arm_id}_link4">
+      <material>Gazebo/White</material>
       <mu1>0.61</mu1>
       <mu2>0.61</mu2>
     </gazebo>
     <gazebo reference="${arm_id}_link5">
+      <material>Gazebo/White</material>
       <mu1>0.61</mu1>
       <mu2>0.61</mu2>
     </gazebo>
     <gazebo reference="${arm_id}_link6">
+      <material>Gazebo/White</material>
       <mu1>0.61</mu1>
       <mu2>0.61</mu2>
     </gazebo>
     <gazebo reference="${arm_id}_link7">
+      <material>Gazebo/White</material>
       <mu1>0.61</mu1>
       <mu2>0.61</mu2>
