Commit message: code

File: mqp_ws/src/scrap_descs/desc/simpleBox.urdf (robot description, URDF)
Before this commit: robot scrap, 2 links, 1 joints
Links:
- link scrap_body: geometry collision mesh filename=package://scrap_descs/desc/mesh/square.dae; visual mesh filename=package://scrap_descs/desc/mesh/square.dae

Commit message: test

File: mqp_ws/src/scrap_descs/desc/simpleBox.urdf (robot description, URDF)
Before this commit: robot scrap, 2 links, 1 joints
Links:
- link scrap_body: geometry collision mesh filename=package://scrap_descs/desc/mesh/square.dae scale=0.3 0.3 0.3; visual mesh filename=package://scrap_descs/desc/mesh/square.dae scale=0.5 0.5 0.5

Commit message: update

File: mqp_ws/src/scrap_descs/desc/simpleBox.urdf (robot description, URDF)
Before this commit: robot scrap, 2 links, 1 joints
Links:
- link scrap_body: geometry collision mesh filename=package://scrap_descs/desc/mesh/square.dae scale=0.3 0.3 0.3; visual mesh filename=package://scrap_descs/desc/mesh/square.dae scale=0.3 0.3 0.3

Commit message: new stuff

File: mqp_ws/src/scrap_descs/desc/simpleBox.urdf (robot description, URDF)
Before this commit: robot scrap, 2 links, 1 joints
Links:
- link scrap_body: geometry collision mesh filename=package://scrap_descs/desc/mesh/square.dae scale=0.5 0.5 0.5; visual mesh filename=package://scrap_descs/desc/mesh/square.dae scale=0.5 0.5 0.5
